File: Hardware/Board.brd (EAGLE design)
At the start: 46 x 35 mm, 105 parts, among them IC1 BQ25180YBGR, IC2 DRV2605YZFR, IC3 BMA421, IC9 RT6160AWSC, J1 TC2030-IDC, J2 503480-2400, J4 KH-TYPE-C-16P, Q1 SI1308EDL-T1-GE3, Q2 20V/4.2A/52mΩ/1.4W, SW1 2025-10-22_07-23-44_LIBRARY_E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

Commit message: Add official submission
Routing:
- net 3V3: track 0.00 -> 192.2 mm, vias 0 -> 26
- net GND: track 0.00 -> 77.5 mm, vias 0 -> 70
- net SDA: track 0.00 -> 76.1 mm, vias 0 -> 6
- net SCL: track 0.00 -> 74.2 mm, vias 0 -> 6
- net VBUS: track 0.00 -> 65.6 mm
- net PREVGH: track 0.00 -> 46.8 mm, vias 0 -> 4
- net SCK: track 0.00 -> 44.4 mm, vias 0 -> 2
- net P0.13: track 0.00 -> 40.7 mm, vias 0 -> 3
- net P1.01: track 0.00 -> 39.8 mm, vias 0 -> 2
- net VREG: track 0.00 -> 38.2 mm
- net EPD_BUSY: track 0.00 -> 38.1 mm, vias 0 -> 2
- net VBAT: track 0.00 -> 36.4 mm, vias 0 -> 2
- net EPD_DC: track 0.00 -> 36.3 mm, vias 0 -> 4
- net EPD_RST: track 0.00 -> 35.7 mm, vias 0 -> 2
- net MOSI: track 0.00 -> 34.3 mm, vias 0 -> 4
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- added copper zone on layer 15, net GND
- added copper zone on layer 2, net GND
- removed copper zone on layer 15, net S$1995
- removed copper zone on layer 2, net S$1996
