File: Hardware/Schematic.sch (EAGLE design)
At the start: 105 parts, among them IC1 BQ25180YBGR, IC2 DRV2605YZFR, IC3 BMA421, IC9 RT6160AWSC, J1 TC2030-IDC, J2 KH-TYPE-C-16P, J3 503480-2400, Q1 SI1308EDL-T1-GE3, Q2 20V/4.2A/52mΩ/1.4W, U1 NRF52840 _QF, U2 MAX17048G+T10, X1 32MHz, X2 32.768kHz

Commit message: Add initial PCB, bill of materials and README
Parts:
- removed J3: 503480-2400, InkTime_v5:503480-2400_503480-2400
- added J4: KH-TYPE-C-16P, InkTime_v5:KH-TYPE-C-16P_KH-TYPE-C-16P
- J2: value KH-TYPE-C-16P -> 503480-2400; device InkTime_v5:KH-TYPE-C-16P_KH-TYPE-C-16P -> InkTime_v5:503480-2400_503480-2400
- renumbered SW_DN to SW3, SW_ENT to SW2, SW_UP to SW1
Connections:
- removed net N$24: C30.1, R5.1, SW1.2
- removed net N$25: C31.1, R8.1, SW2.2
- removed net N$34: C29.1, R7.1, SW3.2
- new net RESE: J2.3, Q1.S, R1_EP_DR.2
- net DN: now also J4.DN1, J4.DN2; no longer J2.DN1, J2.DN2
- net DP: now also J4.DP1, J4.DP2; no longer J2.DP1, J2.DP2
- net EPD_3V3: now also J2.15, J2.16; no longer J3.15, J3.16
- net EPD_BUSY: now also J2.9; no longer J3.9
- net EPD_CS: now also J2.12; no longer J3.12
- net EPD_DC: now also J2.11; no longer J3.11
- net EPD_RST: now also J2.10; no longer J3.10
- net GDR: now also J2.2; no longer J3.2
- net GND: now also J2.17, J2.8, J2.MP1, J2.MP2, J4.GND, J4.SHIELD; no longer J2.GND, J2.SHIELD, J3.17, J3.8, J3.MP1, J3.MP2
- net MOSI: now also J2.14; no longer J3.14
- net N$36: now also J2.24; no longer J3.24
- net N$37: now also J2.18; no longer J3.18
- net N$38: now also J2.19; no longer J3.19
- net N$39: now also J2.20; no longer J3.20
- net N$40: now also J2.21; no longer J3.21
- net N$41: now also J2.22; no longer J3.22
- net N$42: now also J4.CC1; no longer J2.CC1
- net N$44: now also J2.5; no longer J3.5
- net N$45: now also J2.4; no longer J3.4
- net N$47: now also J4.CC2; no longer J2.CC2
- net P0.13: now also C30.1, R5.1, SW1.2
- net P0.14: now also C31.1, R8.1, SW2.2
- net P1.02: now also C29.1, R7.1, SW3.2
- net PREVGL: now also J2.23; no longer J3.23
- net RESET: no longer J3.3, Q1.S, R1_EP_DR.2
- net SCK: now also J2.13; no longer J3.13
- net VBUS: now also J4.VBUS; no longer J2.VBUS

Commit message: Correct electrical schematic as per feedback contents
Parts:
- C25, C33: device InkTime_v5:NORDIC_NRF_3_CAPACITOR_0201_L -> InkTime_v5:NORDIC_NRF_3_CAPACITOR_0402_L
- renumbered C1-EP-DR to C1-EP-DR_0, C2-EP-DR to C2-EP-DR_0, R1_EP_DR to R1_EP_DR_0, R1_USB to R1_USB_0, R2_EP_DR to R2_EP_DR_0, R2_USB to R2_USB_0, R_PWR_EPD to R_PWR_EPD_0, R_TYPE_SEL to R_TYPE_SEL_0, TP_3.3V to TP_3V3_1, TP_3V3 to TP_3V3_0, TP_BAT_GND to TP_BAT_GND_0, TP_GND to TP_GND_0, TP_ON to TP_ON_0, TP_OP to TP_OP_0, TP_RESET to TP_RESET_0, TP_SCL to TP_SCL_0, TP_SDA to TP_SDA_0, TP_SWDCLK to TP_SWDCLK_0, TP_SWDIO to TP_SWDIO_0, TP_SWO to TP_SWO_0, TP_VBAT to TP_VBAT_0, TP_VREG to TP_VREG_0
Connections:
- removed net N$28: C15.2, C16.2, U1.VSS@B7
- net GND: now also C15.2, C16.2, IC9.AGND, IC9.PGND_1, IC9.VSEL, U1.VSS@B7
- net LX1: no longer IC9.AGND, IC9.PGND_1, IC9.VSEL

Commit message: Change switch model value
Parts:
- SW1, SW2, SW3: value 2025-10-22_07-23-44_LIBRARY_EVP-AKE31ASW_EVP-AKE31A_PAN -> EVP-AKE31A
Changed lines of the file:
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@@
 <part name="J2" library="InkTime_v5" library_urn="urn:adsk.wipprod:fs.file:vf.Gd55vp-dRl23AmqAKllygA" deviceset="503480-2400_503480-2400" device="" value="503480-2400"/>
 <part name="U2" library="InkTime_v5" library_urn="urn:adsk.wipprod:fs.file:vf.Gd55vp-dRl23AmqAKllygA" deviceset="ESP32_C6_LIBRARY_MAX17048G+T10" device="" value="MAX17048G+T10"/>
-<part name="SW1" library="InkTime_v5" library_urn="urn:adsk.wipprod:fs.file:vf.Gd55vp-dRl23AmqAKllygA" deviceset="2025-10-22_07-23-44_LIBRARY_EVP-AKE31A" device="SW_EVP-AKE31A_PAN"/>
-<part name="SW2" library="InkTime_v5" library_urn="urn:adsk.wipprod:fs.file:vf.Gd55vp-dRl23AmqAKllygA" deviceset="2025-10-22_07-23-44_LIBRARY_EVP-AKE31A" device="SW_EVP-AKE31A_PAN"/>
-<part name="SW3" library="InkTime_v5" library_urn="urn:adsk.wipprod:fs.file:vf.Gd55vp-dRl23AmqAKllygA" deviceset="2025-10-22_07-23-44_LIBRARY_EVP-AKE31A" device="SW_EVP-AKE31A_PAN"/>
+<part name="SW1" library="InkTime_v5" library_urn="urn:adsk.wipprod:fs.file:vf.Gd55vp-dRl23AmqAKllygA" deviceset="2025-10-22_07-23-44_LIBRARY_EVP-AKE31A" device="SW_EVP-AKE31A_PAN" value="EVP-AKE31A"/>
+<part name="SW2" library="InkTime_v5" library_urn="urn:adsk.wipprod:fs.file:vf.Gd55vp-dRl23AmqAKllygA" deviceset="2025-10-22_07-23-44_LIBRARY_EVP-AKE31A" device="SW_EVP-AKE31A_PAN" value="EVP-AKE31A"/>
+<part name="SW3" library="InkTime_v5" library_urn="urn:adsk.wipprod:fs.file:vf.Gd55vp-dRl23AmqAKllygA" deviceset="2025-10-22_07-23-44_LIBRARY_EVP-AKE31A" device="SW_EVP-AKE31A_PAN" value="EVP-AKE31A"/>
 <part name="EPD_C5" library="InkTime_v5" library_urn="urn:adsk.wipprod:fs.file:vf.Gd55vp-dRl23AmqAKllygA" deviceset="NORDIC_NRF_3_CAPACITOR" device="_0201_L" value="0.1uF/50V"/>
 <part name="SUPPLY58" library="InkTime_v5" library_urn="urn:adsk.wipprod:fs.file:vf.Gd55vp-dRl23AmqAKllygA" deviceset="POWER_SYMBOLS_GND-BAR" device="" value="GND"/>

Commit message: Add official submission
Parts:
- SW3: value EVP-AKE31A -> 2025-10-22_07-23-44_LIBRARY_EVP-AKE31ASW_EVP-AKE31A_PAN
Changed lines of the file:
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@@
 <part name="SW1" library="InkTime_v5" library_urn="urn:adsk.wipprod:fs.file:vf.Gd55vp-dRl23AmqAKllygA" deviceset="2025-10-22_07-23-44_LIBRARY_EVP-AKE31A" device="SW_EVP-AKE31A_PAN" value="EVP-AKE31A"/>
 <part name="SW2" library="InkTime_v5" library_urn="urn:adsk.wipprod:fs.file:vf.Gd55vp-dRl23AmqAKllygA" deviceset="2025-10-22_07-23-44_LIBRARY_EVP-AKE31A" device="SW_EVP-AKE31A_PAN" value="EVP-AKE31A"/>
-<part name="SW3" library="InkTime_v5" library_urn="urn:adsk.wipprod:fs.file:vf.Gd55vp-dRl23AmqAKllygA" deviceset="2025-10-22_07-23-44_LIBRARY_EVP-AKE31A" device="SW_EVP-AKE31A_PAN" value="EVP-AKE31A"/>
+<part name="SW3" library="InkTime_v5" library_urn="urn:adsk.wipprod:fs.file:vf.Gd55vp-dRl23AmqAKllygA" deviceset="2025-10-22_07-23-44_LIBRARY_EVP-AKE31A" device="SW_EVP-AKE31A_PAN"/>
 <part name="EPD_C5" library="InkTime_v5" library_urn="urn:adsk.wipprod:fs.file:vf.Gd55vp-dRl23AmqAKllygA" deviceset="NORDIC_NRF_3_CAPACITOR" device="_0201_L" value="0.1uF/50V"/>
 <part name="SUPPLY58" library="InkTime_v5" library_urn="urn:adsk.wipprod:fs.file:vf.Gd55vp-dRl23AmqAKllygA" deviceset="POWER_SYMBOLS_GND-BAR" device="" value="GND"/>
